File: MainPower.sch (EAGLE design)
At the start: 10 parts, among them IC1 RV-3029-C2

Commit message: Add files via upload
Parts:
- removed DC1: (no value), dc-dc-converter:DC213R
- removed G3: SL-160AA/PR, battery:SL-160AA/PR
- removed IC1: RV-3029-C2, crystal:RV-3029-C2
- removed R2, R3: 10k, rcl:R-EU_0204/2V
- removed U$1: TP4056, TP4056:TP4056
- removed U$3: FRAM, fram:FRAM
- removed U$4: SCD40, SCD40:SCD40
- added C1, C2, C3, C4, C5: 10uF, capacitor-wima:C2,5-3
- added D1: 1N5819-B, diode:1N5819-B
- added G2: SL-340/P3.6V, battery:SL-340/P3.6V
- added L1: (no value), rcl:L-US0204/7
- added LED1: TLLR4400, led:TLLR4400
- added LED2: TLLG4400, led:TLLG4400
- added R1, R10, R4, R5, R6, R7, R8, R9: 1k, rcl:R-EU_0204/2V
- added R11, R12: 10k, rcl:R-EU_0204/2V
- added U1: TP4056, TP4056:TP4056
- added U2: MT3608, MT3608:MT3608
- added U3: DS3231S, DS3231S:DS3231S
- added X1: (no value), con-berg:PN61729
- G1: value SL-160AA/PR -> SL-340/P3.6V; device battery:SL-160AA/PR -> battery:SL-340/P3.6V
Connections:
- removed net N$1: G3.+, IC1.VBACKUP
- new net CLK_RST: U$2.G1, U3.~RST
- new net N$10: R1.2, U1.!CHRG
- new net N$11: C2.1, C3.1, G2.+, L1.1, U1.BAT, U2.EN, U2.IN
- new net N$12: R10.1, R9.2, U2.FB
- new net N$8: LED2.C, R4.2
- new net N$9: LED1.C, R1.1
- new net USB: C1.1, LED1.A, LED2.A, R6.1, R6.2, R8.1, U1.CE, U1.VCC, X1.1
- net 5V: now also C4.1, C5.2, D1.C, R11.1, R12.1, R9.1, U3.VCC; no longer DC1.+VOUT1, IC1.VDD, R2.1, R3.1, U$4.VDD, U$4.VDDH
- net GND: now also C1.2, C2.2, C3.2, C4.2, C5.1, G1.-, G2.-, R10.2, R5.2, R7.1, R7.2, R8.2, U1.GND, U1.TEMP, U2.GND, U3.GND; no longer DC1.-VOUT1, G3.-, IC1.VSS, U$3.GND, U$4.GND
- net N$2: now also D1.A, L1.2, U2.SW; no longer G1.+, U$1.B+
- net N$3: now also R4.1, U1.!STDBY; no longer G1.-, U$1.B-
- net N$4: now also G1.+, U3.VBAT; no longer DC1.-VIN1, U$1.OUT-
- net N$5: now also R5.1, U1.PROG; no longer DC1.+VIN1, U$1.OUT+
- net SCL: now also R11.2, U3.SCL; no longer IC1.SCL, R3.2, U$4.SCL
- net SDA: now also R12.2, U3.SDA; no longer IC1.SDA, R2.2, U$4.SDA
